Commit message: Made Jaws move.

File: jaws_description/urdf/jaws.urdf (robot description, URDF)
Before this commit: robot jaws, 15 links, 14 joints
Links:
- link aft_base: geometry visual box size=0.04 0.02 0.03
- link port_base: geometry visual cylinder length=0.06 radius=0.01
- link stbd_base: geometry visual cylinder length=0.06 radius=0.01
Joints:
- joint aft-body: origin (none) -> xyz=-0.05 0 0 rpy=0 0 0
- joint aft-dome: origin (none) -> xyz=0 0 -0.04 rpy=0 0 0
- joint aft-duct: origin (none) -> xyz=0 0 0.04 rpy=0 0 0
- joint base-aft: origin (none) -> xyz=-0.02 0 0 rpy=0 0 0; parent base_link -> base_endcap
- joint base-dome: origin (none) -> xyz=0.12 0 0 rpy=0 0 0
- joint base-endcap: origin (none) -> xyz=-0.12 0 0 rpy=0 0 0
- joint port-base: axis (none) -> 0 1 0; origin (none) -> xyz=0.06 0.06 0 rpy=0 0 0; type fixed -> continuous
- joint port-body: origin (none) -> xyz=0 0.05 0 rpy=0 0 0
- joint port-dome: origin (none) -> xyz=0 0 -0.04 rpy=0 0 0
- joint port-duct: origin (none) -> xyz=0 0 0.04 rpy=0 0 0
- joint stbd-base: axis (none) -> 0 1 0; origin (none) -> xyz=0.06 -0.06 0 rpy=0 0 0; type fixed -> continuous
- joint stbd-body: origin (none) -> xyz=0 -0.05 0 rpy=0 0 0
- joint stbd-dome: origin (none) -> xyz=0 0 -0.04 rpy=0 0 0
- joint stbd-duct: origin (none) -> xyz=0 0 0.04 rpy=0 0 0

Commit message: One servo is always mounted backwards.

File: jaws_description/urdf/jaws.urdf (robot description, URDF)
Before this commit: robot jaws, 15 links, 14 joints
Joints:
- joint stbd-base: origin xyz=0.06 -0.06 0 rpy=0 0 0 -> xyz=0.06 -0.06 0 rpy=0 0 3.14159
- joint stbd-body: origin xyz=0 -0.05 0 rpy=0 0 0 -> xyz=0 0.05 0 rpy=0 0 0

Commit message: Started using Jaws in Gazebo.

File: jaws_description/urdf/jaws.urdf (robot description, URDF)
Before this commit: robot jaws, 15 links, 14 joints
Links:
- link base_link: mass None -> 1; geometry collision cylinder length=0.24 radius=0.06; visual cylinder length=0.24 radius=0.06
